Commit message: Improved camera position and robotic arm capabilities

File: srdf/ur5_with_gripper.srdf.xacro (robot description, xacro)
@@ -99,4 +99,22 @@
   <disable_collisions link1="wrist_1_link" link2="robotiq_85_left_finger_tip_link" reason="Never" />
   <disable_collisions link1="wrist_1_link" link2="robotiq_85_right_finger_tip_link" reason="Never" />
+  <!-- vs wrist_camera_link -->
+  <disable_collisions link1="wrist_camera_link" link2="wrist_3_link" reason="Adjacent" />
+  <disable_collisions link1="wrist_camera_link" link2="tool0" reason="Adjacent" />
+  <disable_collisions link1="wrist_camera_link" link2="ur_to_robotiq_link" reason="Adjacent" />
+  <disable_collisions link1="wrist_camera_link" link2="robotiq_85_base_link" reason="Never" />
+  <disable_collisions link1="wrist_camera_link" link2="robotiq_85_left_knuckle_link" reason="Never" />
+  <disable_collisions link1="wrist_camera_link" link2="robotiq_85_right_knuckle_link" reason="Never" />
+  <disable_collisions link1="wrist_camera_link" link2="robotiq_85_left_inner_knuckle_link" reason="Never" />
+  <disable_collisions link1="wrist_camera_link" link2="robotiq_85_right_inner_knuckle_link" reason="Never" />
+  <disable_collisions link1="wrist_camera_link" link2="robotiq_85_left_finger_link" reason="Never" />
+  <disable_collisions link1="wrist_camera_link" link2="robotiq_85_right_finger_link" reason="Never" />
+  <disable_collisions link1="wrist_camera_link" link2="robotiq_85_left_finger_tip_link" reason="Never" />
+  <disable_collisions link1="wrist_camera_link" link2="robotiq_85_right_finger_tip_link" reason="Never" />
+  <disable_collisions link1="wrist_camera_link" link2="wrist_2_link" reason="Never" />
+  <disable_collisions link1="wrist_camera_link" link2="wrist_1_link" reason="Never" />
+  <disable_collisions link1="wrist_camera_link" link2="forearm_link" reason="Never" />
+  <disable_collisions link1="wrist_camera_link" link2="upper_arm_link" reason="Never" />
+  <disable_collisions link1="wrist_camera_link" link2="shoulder_link" reason="Never" />
   <!-- vs forearm_link -->
   <disable_collisions link1="forearm_link" link2="ur_to_robotiq_link" reason="Never" />

File: urdf/ur5_with_gripper.urdf.xacro (robot description, xacro)
@@ -119,5 +119,5 @@
     <inertial>
       <mass value="0.05"/>
-      <inertia ixx="0.0001" iyy="0.0001" izz="0.0001"/>
+      <inertia ixx="0.0001" ixy="0" ixz="0" iyy="0.0001" iyz="0" izz="0.0001"/>
     </inertial>
   </link>
@@ -125,5 +125,5 @@
     <parent link="tool0"/>
     <child link="wrist_camera_link"/>
-    <origin xyz="0 -0.04 -0.01" rpy="0 -1.5708 0"/>
+    <origin xyz="0 -0.05 -0.01" rpy="0 -1.5708 0"/>
   </joint>
   <link name="wrist_camera_optical_link"/>
